Commit message: Modified f1 f2 collision meshes

File: cyclo_motion_controller_models/models/ai_worker/ffw_f1_follower.urdf (robot description, URDF)
Before this commit: robot ffw_f1_follower, 18 links, 17 joints
Links:
- added link head_link1
- added link head_link2; collision sphere radius=0.1
- link arm_base_link: geometry collision box size=0.2 0.1 0.63; collision box size=0.2 0.1 0.63
- link arm_l_link1: geometry 
- link arm_l_link2: geometry collision cylinder length=0.32 radius=0.07; collision sphere radius=0.07
- link arm_l_link3: geometry 
- link arm_l_link4: geometry collision cylinder length=0.2785 radius=0.07; collision sphere radius=0.07
- link arm_l_link5: geometry 
- link arm_l_link6: geometry 
- link arm_l_link7: geometry collision cylinder length=0.091 radius=0.085; collision sphere radius=0.085
- link arm_r_link1: geometry 
- link arm_r_link2: geometry collision cylinder length=0.32 radius=0.07; collision sphere radius=0.07
- link arm_r_link3: geometry 
- link arm_r_link4: geometry collision cylinder length=0.2785 radius=0.07; collision sphere radius=0.07
- link arm_r_link5: geometry 
- link arm_r_link6: geometry 
- link arm_r_link7: geometry collision cylinder length=0.091 radius=0.085; collision sphere radius=0.085
- link end_effector_l_link: geometry visual box size=0.01 0.01 0.01
- link end_effector_r_link: geometry visual box size=0.01 0.01 0.01
Joints:
- added joint head_joint1: type fixed, parent arm_base_link, child head_link1, origin xyz=0.102729 0 0.132803 rpy=0 0 0
- added joint head_joint2: type fixed, parent head_link1, child head_link2, origin xyz=0.0141410 0 0.0555070 rpy=0 0 0

File: cyclo_motion_controller_models/models/ai_worker/ffw_f2_follower.urdf (robot description, URDF)
Before this commit: robot ffw_f2_follower, 18 links, 17 joints
Links:
- added link head_link1
- added link head_link2; collision sphere radius=0.1
- link arm_base_link: geometry collision box size=0.2 0.1 0.63; collision box size=0.2 0.1 0.63
- link arm_l_link1: geometry 
- link arm_l_link2: geometry collision cylinder length=0.32 radius=0.07; collision sphere radius=0.07
- link arm_l_link3: geometry 
- link arm_l_link4: geometry collision cylinder length=0.2785 radius=0.07; collision sphere radius=0.07
- link arm_l_link5: geometry 
- link arm_l_link6: geometry 
- link arm_l_link7: geometry collision cylinder length=0.091 radius=0.085; collision sphere radius=0.085
- link arm_r_link1: geometry 
- link arm_r_link2: geometry collision cylinder length=0.32 radius=0.07; collision sphere radius=0.07
- link arm_r_link3: geometry 
- link arm_r_link4: geometry collision cylinder length=0.2785 radius=0.07; collision sphere radius=0.07
- link arm_r_link5: geometry 
- link arm_r_link6: geometry 
- link arm_r_link7: geometry collision cylinder length=0.091 radius=0.085; collision sphere radius=0.085
- link end_effector_l_link: geometry visual box size=0.01 0.01 0.01
- link end_effector_r_link: geometry visual box size=0.01 0.01 0.01
Joints:
- added joint head_joint1: type fixed, parent arm_base_link, child head_link1, origin xyz=0.102729 0 0.132803 rpy=0 0 0
- added joint head_joint2: type fixed, parent head_link1, child head_link2, origin xyz=0.0141410 0 0.0555070 rpy=0 0 0

Commit message: Update AI Worker follower models and RViz launch support

File: cyclo_motion_controller_models/models/ai_worker/ffw_f1_follower.urdf (robot description, URDF)
Before this commit: robot ffw_f1_follower, 20 links, 19 joints
Links:
- link arm_base_link: geometry collision box size=0.2 0.1 0.63; collision box size=0.2 0.1 0.63
- link arm_l_link1: geometry visual mesh filename=package://ffw_description/meshes/common/follower/ffw_f/arm_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 scale=0.001 0.001 0.001
- link arm_l_link2: geometry collision cylinder length=0.32 radius=0.07; collision sphere radius=0.07
- link arm_l_link3: geometry visual mesh filename=package://ffw_description/meshes/common/follower/ffw_f/arm_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 scale=0.001 0.001 0.001
- link arm_l_link4: geometry collision cylinder length=0.2785 radius=0.07; collision sphere radius=0.07
- link arm_l_link5: geometry visual mesh filename=package://ffw_description/meshes/common/follower/ffw_f/arm_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 scale=0.001 0.001 0.001
- link arm_l_link6: geometry visual mesh filename=package://ffw_description/meshes/common/follower/ffw_f/arm_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 scale=0.001 0.001 0.001
- link arm_l_link7: geometry collision cylinder length=0.091 radius=0.085; collision sphere radius=0.085
- link arm_r_link1: geometry visual mesh filename=package://ffw_description/meshes/common/follower/ffw_f/arm_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 scale=0.001 0.001 0.001
- link arm_r_link2: geometry collision cylinder length=0.32 radius=0.07; collision sphere radius=0.07
- link arm_r_link3: geometry visual mesh filename=package://ffw_description/meshes/common/follower/ffw_f/arm_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 scale=0.001 0.001 0.001
- link arm_r_link4: geometry collision cylinder length=0.2785 radius=0.07; collision sphere radius=0.07
- link arm_r_link5: geometry visual mesh filename=package://ffw_description/meshes/common/follower/ffw_f/arm_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 scale=0.001 0.001 0.001
- link arm_r_link6: geometry visual mesh filename=package://ffw_description/meshes/common/follower/ffw_f/arm_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 scale=0.001 0.001 0.001
- link arm_r_link7: geometry collision cylinder length=0.091 radius=0.085; collision sphere radius=0.085
- link base_link: geometry collision box size=0.6 0.4 0.3; collision cylinder length=0.4 radius=0.15
- link head_link1: geometry visual mesh filename=package://ffw_description/meshes/common/follower/ffw_f/head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 scale=0.001 0.001 0.001
- link head_link2: geometry collision sphere radius=0.1; visual mesh filename=package://ffw_description/meshes/common/follower/ffw_f/head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 scale=0.001 0.001 0.001
Joints:
- joint arm_l_joint1: origin xyz=0.059 0.1127 0.030 rpy=0 0 0 -> xyz=0.0555 0.11345 0.014 rpy=0 0 0
- joint arm_l_joint2: origin xyz=0.0177 0.1038 0 rpy=0 0 0 -> xyz=0.01845 0.10305 0 rpy=0 0 0
- joint arm_l_joint3: origin xyz=-0.0177 0 -0.2072 rpy=0 0 0 -> xyz=-0.01845 0 -0.20795 rpy=0 0 0
- joint arm_l_joint4: limit lower=-2.9361 upper=1.0786 effort=1000 velocity=4.8 -> lower=-2.9361 upper=-0.7 effort=1000 velocity=4.8; origin xyz=0.0410041 0.0007 -0.1128 rpy=0 0 0 -> xyz=0.0410041 0.00145 -0.11205 rpy=0 0 0
- joint arm_l_joint5: origin xyz=-0.041 -0.0007 -0.1477 rpy=0 0 0 -> xyz=-0.041 -0.00145 -0.14845 rpy=0 0 0
- joint arm_l_joint6: origin xyz=0 0.0007 -0.0948 rpy=0 0 0 -> xyz=0 0.00145 -0.09405 rpy=0 0 0
- joint arm_l_joint7: origin xyz=-0.00025 -0.0007 -0.0775 rpy=0 0 0 -> xyz=-0.00025 -0.00145 -0.0775 rpy=0 0 0
- joint arm_r_joint1: origin xyz=0.055 -0.1127 0.030 rpy=0 0 0 -> xyz=0.0555 -0.11345 0.014 rpy=0 0 0
- joint arm_r_joint2: origin xyz=0.0177 -0.1038 0 rpy=0 0 0 -> xyz=0.01845 -0.10305 0 rpy=0 0 0
- joint arm_r_joint3: origin xyz=-0.0177 0 -0.2072 rpy=0 0 0 -> xyz=-0.01845 0 -0.20795 rpy=0 0 0
- joint arm_r_joint4: limit lower=-2.9361 upper=1.0786 effort=1000 velocity=4.8 -> lower=-2.9361 upper=-0.7 effort=1000 velocity=4.8; origin xyz=0.0410041 -0.0007 -0.1128 rpy=0 0 0 -> xyz=0.0410041 -0.00145 -0.11205 rpy=0 0 0
- joint arm_r_joint5: origin xyz=-0.041 0.0007 -0.1477 rpy=0 0 0 -> xyz=-0.041 0.00145 -0.14845 rpy=0 0 0
- joint arm_r_joint6: origin xyz=0 -0.0007 -0.0948 rpy=0 0 0 -> xyz=0 -0.00145 -0.09405 rpy=0 0 0
- joint arm_r_joint7: origin xyz=-0.00025 -0.0007 -0.0775 rpy=0 0 0 -> xyz=-0.00025 -0.00145 -0.0775 rpy=0 0 0
- joint head_joint1: origin xyz=0.102729 0 0.132803 rpy=0 0 0 -> xyz=0.102729 0 0.116803 rpy=0 0 0
- joint head_joint2: origin xyz=0.0141410 0 0.0555070 rpy=0 0 0 -> xyz=0.04 0 0.064 rpy=0 0 0
- joint lift_joint: origin xyz=0.0055 0 1.4316 rpy=0 0 0 -> xyz=-0.05 0 1.4166 rpy=0 0 0

File: cyclo_motion_controller_models/models/ai_worker/ffw_f2_follower.urdf (robot description, URDF)
Before this commit: robot ffw_f2_follower, 20 links, 19 joints
Links:
- link arm_base_link: geometry collision box size=0.2 0.1 0.63; collision box size=0.2 0.1 0.63
- link arm_l_link1: geometry visual mesh filename=package://ffw_description/meshes/common/follower/ffw_f/arm_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 scale=0.001 0.001 0.001
- link arm_l_link2: geometry collision cylinder length=0.32 radius=0.07; collision sphere radius=0.07
- link arm_l_link3: geometry visual mesh filename=package://ffw_description/meshes/common/follower/ffw_f/arm_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 scale=0.001 0.001 0.001
- link arm_l_link4: geometry collision cylinder length=0.2785 radius=0.07; collision sphere radius=0.07
- link arm_l_link5: geometry visual mesh filename=package://ffw_description/meshes/common/follower/ffw_f/arm_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 scale=0.001 0.001 0.001
- link arm_l_link6: geometry visual mesh filename=package://ffw_description/meshes/common/follower/ffw_f/arm_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 scale=0.001 0.001 0.001
- link arm_l_link7: geometry collision cylinder length=0.091 radius=0.085; collision sphere radius=0.085
- link arm_r_link1: geometry visual mesh filename=package://ffw_description/meshes/common/follower/ffw_f/arm_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 scale=0.001 0.001 0.001
- link arm_r_link2: geometry collision cylinder length=0.32 radius=0.07; collision sphere radius=0.07
- link arm_r_link3: geometry visual mesh filename=package://ffw_description/meshes/common/follower/ffw_f/arm_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 scale=0.001 0.001 0.001
- link arm_r_link4: geometry collision cylinder length=0.2785 radius=0.07; collision sphere radius=0.07
- link arm_r_link5: geometry visual mesh filename=package://ffw_description/meshes/common/follower/ffw_f/arm_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 scale=0.001 0.001 0.001
- link arm_r_link6: geometry visual mesh filename=package://ffw_description/meshes/common/follower/ffw_f/arm_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 scale=0.001 0.001 0.001
- link arm_r_link7: geometry collision cylinder length=0.091 radius=0.085; collision sphere radius=0.085
- link base_link: geometry collision box size=0.6 0.4 0.3; collision cylinder length=0.4 radius=0.15
- link head_link1: geometry visual mesh filename=package://ffw_description/meshes/common/follower/ffw_f/head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 scale=0.001 0.001 0.001
- link head_link2: geometry collision sphere radius=0.1; visual mesh filename=package://ffw_description/meshes/common/follower/ffw_f/head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 scale=0.001 0.001 0.001
Joints:
- joint arm_l_joint1: origin xyz=0.059 0.1127 0.030 rpy=0 0 0 -> xyz=0.0555 0.11345 0.014 rpy=0 0 0
- joint arm_l_joint2: origin xyz=0.0177 0.1038 0 rpy=0 0 0 -> xyz=0.01845 0.10305 0 rpy=0 0 0
- joint arm_l_joint3: origin xyz=-0.0177 0 -0.2072 rpy=0 0 0 -> xyz=-0.01845 0 -0.20795 rpy=0 0 0
- joint arm_l_joint4: limit lower=-2.9361 upper=1.0786 effort=1000 velocity=4.8 -> lower=-2.9361 upper=-0.7 effort=1000 velocity=4.8; origin xyz=0.0410041 0.0007 -0.1128 rpy=0 0 0 -> xyz=0.0410041 0.00145 -0.11205 rpy=0 0 0
- joint arm_l_joint5: origin xyz=-0.041 -0.0007 -0.1477 rpy=0 0 0 -> xyz=-0.041 -0.00145 -0.14845 rpy=0 0 0
- joint arm_l_joint6: origin xyz=0 0.0007 -0.0948 rpy=0 0 0 -> xyz=0 0.00145 -0.09405 rpy=0 0 0
- joint arm_l_joint7: origin xyz=-0.00025 -0.0007 -0.0775 rpy=0 0 0 -> xyz=-0.00025 -0.00145 -0.0775 rpy=0 0 0
- joint arm_r_joint1: origin xyz=0.055 -0.1127 0.030 rpy=0 0 0 -> xyz=0.0555 -0.11345 0.014 rpy=0 0 0
- joint arm_r_joint2: origin xyz=0.0177 -0.1038 0 rpy=0 0 0 -> xyz=0.01845 -0.10305 0 rpy=0 0 0
- joint arm_r_joint3: origin xyz=-0.0177 0 -0.2072 rpy=0 0 0 -> xyz=-0.01845 0 -0.20795 rpy=0 0 0
- joint arm_r_joint4: limit lower=-2.9361 upper=1.0786 effort=1000 velocity=4.8 -> lower=-2.9361 upper=-0.7 effort=1000 velocity=4.8; origin xyz=0.0410041 -0.0007 -0.1128 rpy=0 0 0 -> xyz=0.0410041 -0.00145 -0.11205 rpy=0 0 0
- joint arm_r_joint5: origin xyz=-0.041 0.0007 -0.1477 rpy=0 0 0 -> xyz=-0.041 0.00145 -0.14845 rpy=0 0 0
- joint arm_r_joint6: origin xyz=0 -0.0007 -0.0948 rpy=0 0 0 -> xyz=0 -0.00145 -0.09405 rpy=0 0 0
- joint arm_r_joint7: origin xyz=-0.00025 -0.0007 -0.0775 rpy=0 0 0 -> xyz=-0.00025 -0.00145 -0.0775 rpy=0 0 0
- joint head_joint1: origin xyz=0.102729 0 0.132803 rpy=0 0 0 -> xyz=0.102729 0 0.116803 rpy=0 0 0
- joint head_joint2: origin xyz=0.0141410 0 0.0555070 rpy=0 0 0 -> xyz=0.04 0 0.064 rpy=0 0 0
- joint lift_joint: origin xyz=-0.0753807 0 1.407 rpy=0 0 0 -> xyz=-0.075 0 1.423 rpy=0 0 0
