Commit message: Update a1 urdf and modify rviz config file

File: cyclo_motion_controller_models/models/ai_worker/leader/ffw_a1_leader.urdf (robot description, URDF)
Before this commit: robot ffw_a1_leader, 18 links, 17 joints
Joints:
- joint arm_l_joint1: axis 0 1 0 -> 1 0 0; origin xyz=0 0.13070 0 rpy=0 0 0 -> xyz=0 0.1912 0 rpy=0 0 0
- joint arm_l_joint2: axis 1 0 0 -> 0 1 0; origin xyz=0 0.042 0 rpy=0 0 0 -> xyz=0.120795 0.0795 -0.000151884 rpy=0 0 0
- joint arm_l_joint3: origin xyz=0 0 -0.108 rpy=0 0 0 -> xyz=-0.00005 0 -0.2295 rpy=0 0 0
- joint arm_l_joint4: origin xyz=0.01642 0 -0.04151 rpy=0 0 0 -> xyz=0 0 0 rpy=0 0 0
- joint arm_l_joint5: origin xyz=-0.01642 0 -0.07802 rpy=0 0 0 -> xyz=-0.036 0 -0.21345 rpy=0 0 0
- joint arm_l_joint6: origin xyz=0 0 -0.044 rpy=0 0 0 -> xyz=0 0 0 rpy=0 0 0
- joint arm_l_joint7: origin xyz=0 0 -0.0275 rpy=0 0 0 -> xyz=0.0796388 -0.07945 0.0001 rpy=0 0 0
- joint arm_r_joint1: axis 0 1 0 -> 1 0 0; origin xyz=0 -0.13070 0 rpy=0 0 0 -> xyz=0 -0.1912 0 rpy=0 0 0
- joint arm_r_joint2: axis 1 0 0 -> 0 1 0; origin xyz=0 -0.042 0 rpy=0 0 0 -> xyz=0.120795198 -0.0795 -0.000251884 rpy=0 0 0
- joint arm_r_joint3: origin xyz=0 0 -0.108 rpy=0 0 0 -> xyz=-0.00005 0 -0.2295 rpy=0 0 0
- joint arm_r_joint4: origin xyz=0.01642 0 -0.04151 rpy=0 0 0 -> xyz=0 0 0 rpy=0 0 0
- joint arm_r_joint5: origin xyz=-0.01642 0 -0.07802 rpy=0 0 0 -> xyz=-0.036 0 -0.21355 rpy=0 0 0
- joint arm_r_joint6: origin xyz=0 0 -0.044 rpy=0 0 0 -> xyz=0 0 0 rpy=0 0 0
- joint arm_r_joint7: origin xyz=0 0 -0.0275 rpy=0 0 0 -> xyz=0.0796388 0.07945 0 rpy=0 0 0
- joint end_effector_l_joint: origin xyz=0 0 -0.186 rpy=0 0 0 -> xyz=0 0 0 rpy=0 0 0
- joint end_effector_r_joint: origin xyz=0 0 -0.186 rpy=0 0 0 -> xyz=0 0 0 rpy=0 0 0

Commit message: Modified a1 eef position

File: cyclo_motion_controller_models/models/ai_worker/leader/ffw_a1_leader.urdf (robot description, URDF)
Before this commit: robot ffw_a1_leader, 18 links, 17 joints
Joints:
- joint end_effector_l_joint: origin xyz=0 0 0 rpy=0 0 0 -> xyz=0 0 -0.15 rpy=0 0 0
- joint end_effector_r_joint: origin xyz=0 0 0 rpy=0 0 0 -> xyz=0 0 -0.15 rpy=0 0 0
